Commit message: biped model v2

File: biped_model.urdf (robot description, URDF)
Before this commit: robot no, 37 links, 36 joints
Links:
- link base_link: mass 6.458470839830133 -> 6.087495213581755
- link servo_v11: mass 0.25257832542625036 -> 0.2525811539773393
- link servo_v1_101: mass 0.25257832542625036 -> 0.2525811539773393
- link servo_v1_111: mass 0.25257832542625036 -> 0.2525811539773393
- link servo_v1_21: mass 0.25257832542625036 -> 0.2525811539773393
- link servo_v1_31: mass 0.25257832542625036 -> 0.2525811539773393
- link servo_v1_41: mass 0.25257832542625036 -> 0.2525811539773393
- link servo_v1_51: mass 0.25257832542625036 -> 0.2525811539773393
- link servo_v1_61: mass 0.25257832542625036 -> 0.2525811539773393
- link servo_v1_71: mass 0.25257832542625036 -> 0.2525811539773393
- link servo_v1_81: mass 0.25257832542625036 -> 0.2525811539773393
- link servo_v1_91: mass 0.25257832542625036 -> 0.2525811539773393
Joints:
- removed joint Rigid10
- removed joint Rigid5
- removed joint Rigid6
- removed joint Rigid9
- added joint Rigid53: type fixed, parent darwin_SP0-5_Dfaut_v11, child puru_returns_Component6_v31, origin xyz=0.0 0.0 0.006 rpy=0 0 0
- added joint Rigid55: type fixed, parent darwin_SP0-5_Dfaut_v1_11, child puru_returns_Component6_v3_11, origin xyz=0.0 0.0 0.006 rpy=0 0 0
- added joint Rigid56: type fixed, parent base_link, child servo_v11, origin xyz=-0.006829 -0.137658 -0.013403 rpy=0 0 0
- added joint Rigid57: type fixed, parent base_link, child servo_v1_11, origin xyz=0.104916 -0.137658 -0.013403 rpy=0 0 0
- joint Rev12: origin xyz=-0.006959 0.052255 -0.1881 rpy=0 0 0 -> xyz=-0.006955 0.031899 -0.1881 rpy=0 0 0
- joint Rev14: origin xyz=0.093041 0.052255 -0.1881 rpy=0 0 0 -> xyz=0.093045 0.031899 -0.1881 rpy=0 0 0
- joint Rev18: origin xyz=-0.000399 0.009753 0.183731 rpy=0 0 0 -> xyz=0.019956 0.009749 0.183732 rpy=0 0 0
- joint Rev21: origin xyz=-0.064725 0.021121 -0.063307 rpy=0 0 0 -> xyz=-0.064725 -0.01959 -0.063298 rpy=0 0 0
- joint Rev24: origin xyz=0.410911 -0.0357 0.001939 rpy=0 0 0 -> xyz=0.41091 -0.035695 0.022295 rpy=0 0 0
- joint Rev39: origin xyz=-0.02811 -0.307804 0.370192 rpy=0 0 0 -> xyz=-0.028111 -0.348515 0.370201 rpy=0 0 0
- joint Rev42: origin xyz=0.772672 0.03081 -0.129401 rpy=0 0 0 -> xyz=0.772672 0.010455 -0.129406 rpy=0 0 0
- joint Rev46: origin xyz=0.032684 -0.057488 -0.018743 rpy=0 0 0 -> xyz=0.053035 -0.077849 -0.018744 rpy=0 0 0
- joint Rev7: origin xyz=-0.005875 -0.01631 -0.034578 rpy=0 0 0 -> xyz=-0.00587 -0.01631 0.034578 rpy=0 0 0
- joint Rev8: origin xyz=0.00587 -0.01631 -0.034578 rpy=0 0 0 -> xyz=0.005875 -0.01631 0.034578 rpy=0 0 0
- joint Rigid11: origin xyz=0.0 -0.035632 -0.056073 rpy=0 0 0 -> xyz=0.006 -0.035632 -0.062074 rpy=0 0 0
- joint Rigid13: origin xyz=0.0 -0.035632 -0.056073 rpy=0 0 0 -> xyz=0.006 -0.035632 -0.062074 rpy=0 0 0
- joint Rigid16: origin xyz=-0.033619 -0.046385 0.20616 rpy=0 0 0 -> xyz=-0.033623 -0.026029 0.20616 rpy=0 0 0
- joint Rigid19: origin xyz=-0.014911 -0.023976 -0.195601 rpy=0 0 0 -> xyz=-0.035266 -0.023972 -0.195602 rpy=0 0 0
- joint Rigid20: origin xyz=0.365635 -0.132869 0.039112 rpy=0 0 0 -> xyz=0.365635 -0.112513 0.039108 rpy=0 0 0
- joint Rigid22: origin xyz=-0.2846 0.016162 0.036024 rpy=0 0 0 -> xyz=-0.2846 0.036517 0.036019 rpy=0 0 0
- joint Rigid26: origin xyz=0.009611 -0.076448 0.40759 rpy=0 0 0 -> xyz=0.009615 -0.056093 0.407589 rpy=0 0 0
- joint Rigid28: origin xyz=-0.007833 0.01993 -0.424031 rpy=0 0 0 -> xyz=-0.007837 -0.000425 -0.424031 rpy=0 0 0
- joint Rigid29: origin xyz=-0.394601 0.064277 0.003935 rpy=0 0 0 -> xyz=-0.3946 0.064272 -0.01642 rpy=0 0 0
- joint Rigid35: origin xyz=-0.064463 -0.04638 0.20441 rpy=0 0 0 -> xyz=-0.064468 -0.026024 0.20441 rpy=0 0 0
- joint Rigid36: origin xyz=-0.017693 0.00835 0.0333 rpy=0 0 0 -> xyz=-0.017692 0.00835 0.033301 rpy=0 0 0
- joint Rigid38: origin xyz=0.326016 0.19181 -0.243377 rpy=0 0 0 -> xyz=0.326016 0.212166 -0.243382 rpy=0 0 0
- joint Rigid40: origin xyz=-0.314216 0.014407 -0.132726 rpy=0 0 0 -> xyz=-0.314215 0.034762 -0.13273 rpy=0 0 0
- joint Rigid41: origin xyz=-0.759816 -0.155032 0.135276 rpy=0 0 0 -> xyz=-0.759817 -0.134677 0.13528 rpy=0 0 0
- joint Rigid43: origin xyz=-0.01631 0.036293 0.007081 rpy=0 0 0 -> xyz=-0.01631 0.036293 0.007082 rpy=0 0 0
- joint Rigid44: origin xyz=-0.057288 -0.076992 0.40587 rpy=0 0 0 -> xyz=-0.057283 -0.056636 0.40587 rpy=0 0 0
- joint Rigid47: origin xyz=0.049182 0.105962 -0.423311 rpy=0 0 0 -> xyz=0.028826 0.105967 -0.423311 rpy=0 0 0

Commit message: fixed biped model

File: biped_model.urdf (robot description, URDF)
Before this commit: robot COM, 37 links, 36 joints
Links:
- removed link New_Component_v21Component171
- removed link New_Component_v2_11Component311
- removed link New_comp_mirror_v11
- removed link New_comp_v31
- removed link darwin_SP0-5_Dfaut_v11
- removed link darwin_SP0-5_Dfaut_v1_11
- removed link darwin_SP0-5_Dfaut_v1_111
- removed link darwin_SP0-5_Dfaut_v1_121
- removed link darwin_SP0-5_Dfaut_v1_21
- removed link darwin_SP0-5_Dfaut_v1_31
- removed link darwin_SP0-5_Dfaut_v1_41
- removed link darwin_SP0-5_Dfaut_v1_51
- removed link darwin_SP0-5_Dfaut_v1_61
- removed link darwin_SP0-5_Dfaut_v1_71
- removed link darwin_SP0-5_Dfaut_v1_81
- removed link darwin_SP0-5_Dfaut_v1_91
- removed link puru_returns_Component1_mirror_v11
- removed link puru_returns_Component1_v21
- removed link puru_returns_Component3_Copy_mirror_v11
- removed link puru_returns_Component3_Copy_v11
- removed link puru_returns_Component6_v31
- removed link puru_returns_Component6_v3_11
- removed link servo_v11
- removed link servo_v1_101
- removed link servo_v1_11
- removed link servo_v1_111
- removed link servo_v1_21
- removed link servo_v1_31
- removed link servo_v1_41
- removed link servo_v1_51
- removed link servo_v1_61
- removed link servo_v1_71
- removed link servo_v1_81
- removed link servo_v1_91
- removed link testing_Component2_Copy_v11Component241
- removed link testing_Component2__mirror_v11
- added link ComponentL11, mass 0.04702613835521159; collision mesh filename=meshes1/ComponentL11.stl scale=0.001 0.001 0.001; visual mesh filename=meshes1/ComponentL11.stl scale=0.001 0.001 0.001
- added link ComponentL21, mass 0.09272661140293512; collision mesh filename=meshes1/ComponentL21.stl scale=0.001 0.001 0.001; visual mesh filename=meshes1/ComponentL21.stl scale=0.001 0.001 0.001
- added link ComponentL31Component311, mass 0.12057690606604259; collision mesh filename=meshes1/ComponentL31Component311.stl scale=0.001 0.001 0.001; visual mesh filename=meshes1/ComponentL31Component311.stl scale=0.001 0.001 0.001
- added link ComponentL41, mass 0.1851062904404302; collision mesh filename=meshes1/ComponentL41.stl scale=0.001 0.001 0.001; visual mesh filename=meshes1/ComponentL41.stl scale=0.001 0.001 0.001
- added link ComponentL51, mass 0.08459586965507518; collision mesh filename=meshes1/ComponentL51.stl scale=0.001 0.001 0.001; visual mesh filename=meshes1/ComponentL51.stl scale=0.001 0.001 0.001
- added link ComponentL61, mass 0.3521119210080811; collision mesh filename=meshes1/ComponentL61.stl scale=0.001 0.001 0.001; visual mesh filename=meshes1/ComponentL61.stl scale=0.001 0.001 0.001
- added link ComponentR11, mass 0.04762273835521005; collision mesh filename=meshes1/ComponentR11.stl scale=0.001 0.001 0.001; visual mesh filename=meshes1/ComponentR11.stl scale=0.001 0.001 0.001
- added link ComponentR21, mass 0.09185709979828287; collision mesh filename=meshes1/ComponentR21.stl scale=0.001 0.001 0.001; visual mesh filename=meshes1/ComponentR21.stl scale=0.001 0.001 0.001
- added link ComponentR31Component171, mass 0.12406261058924599; collision mesh filename=meshes1/ComponentR31Component171.stl scale=0.001 0.001 0.001; visual mesh filename=meshes1/ComponentR31Component171.stl scale=0.001 0.001 0.001
- added link ComponentR41, mass 0.18510629044043106; collision mesh filename=meshes1/ComponentR41.stl scale=0.001 0.001 0.001; visual mesh filename=meshes1/ComponentR41.stl scale=0.001 0.001 0.001
- added link ComponentR51Component241, mass 0.08459587295154185; collision mesh filename=meshes1/ComponentR51Component241.stl scale=0.001 0.001 0.001; visual mesh filename=meshes1/ComponentR51Component241.stl scale=0.001 0.001 0.001
- added link ComponentR61, mass 0.3521119210080813; collision mesh filename=meshes1/ComponentR61.stl scale=0.001 0.001 0.001; visual mesh filename=meshes1/ComponentR61.stl scale=0.001 0.001 0.001
- added link ServoL21, mass 0.2525811539773393; collision mesh filename=meshes1/ServoL21.stl scale=0.001 0.001 0.001; visual mesh filename=meshes1/ServoL21.stl scale=0.001 0.001 0.001
- added link ServoL41, mass 0.2525811539773393; collision mesh filename=meshes1/ServoL41.stl scale=0.001 0.001 0.001; visual mesh filename=meshes1/ServoL41.stl scale=0.001 0.001 0.001
- added link ServoL51, mass 0.2525811539773393; collision mesh filename=meshes1/ServoL51.stl scale=0.001 0.001 0.001; visual mesh filename=meshes1/ServoL51.stl scale=0.001 0.001 0.001
- added link ServoL61, mass 0.2525811539773393; collision mesh filename=meshes1/ServoL61.stl scale=0.001 0.001 0.001; visual mesh filename=meshes1/ServoL61.stl scale=0.001 0.001 0.001
- added link ServoR41, mass 0.2525811539773393; collision mesh filename=meshes1/ServoR41.stl scale=0.001 0.001 0.001; visual mesh filename=meshes1/ServoR41.stl scale=0.001 0.001 0.001
- added link ServoR61, mass 0.2525811539773393; collision mesh filename=meshes1/ServoR61.stl scale=0.001 0.001 0.001; visual mesh filename=meshes1/ServoR61.stl scale=0.001 0.001 0.001
- added link servoL11, mass 0.25257832542625036; collision mesh filename=meshes1/servoL11.stl scale=0.001 0.001 0.001; visual mesh filename=meshes1/servoL11.stl scale=0.001 0.001 0.001
- added link servoL31, mass 0.2525811539773393; collision mesh filename=meshes1/servoL31.stl scale=0.001 0.001 0.001; visual mesh filename=meshes1/servoL31.stl scale=0.001 0.001 0.001
- added link servoR1v11, mass 0.2525811539773393; collision mesh filename=meshes1/servoR1v11.stl scale=0.001 0.001 0.001; visual mesh filename=meshes1/servoR1v11.stl scale=0.001 0.001 0.001
- added link servoR21, mass 0.2525811539773393; collision mesh filename=meshes1/servoR21.stl scale=0.001 0.001 0.001; visual mesh filename=meshes1/servoR21.stl scale=0.001 0.001 0.001
- added link servoR31, mass 0.2525811539773393; collision mesh filename=meshes1/servoR31.stl scale=0.001 0.001 0.001; visual mesh filename=meshes1/servoR31.stl scale=0.001 0.001 0.001
- added link servoR51, mass 0.2525811539773393; collision mesh filename=meshes1/servoR51.stl scale=0.001 0.001 0.001; visual mesh filename=meshes1/servoR51.stl scale=0.001 0.001 0.001
- link base_link: geometry collision mesh filename=meshes1/base_link.stl scale=0.001 0.001 0.001; visual mesh filename=meshes1/base_link.stl scale=0.001 0.001 0.001
Joints:
- removed joint Rev12
- removed joint Rev14
- removed joint Rev18
- removed joint Rev21
- removed joint Rev24
- removed joint Rev27
- removed joint Rev33
- removed joint Rev39
- removed joint Rev42
- removed joint Rev46
- removed joint Rev7
- removed joint Rev8
- removed joint Rigid11
- removed joint Rigid13
- removed joint Rigid17
- removed joint Rigid19
- removed joint Rigid20
- removed joint Rigid23
- removed joint Rigid26
- removed joint Rigid38
- removed joint Rigid41
- removed joint Rigid44
- removed joint Rigid45
- removed joint Rigid47
- removed joint Rigid53
- removed joint Rigid55
- added joint Rev68: type continuous, parent servoR1v11, child ComponentR11, origin xyz=0.005875 -0.01631 0.034578 rpy=0 0 0, axis -0.0 -1.0 0.0
- added joint Rev69: type continuous, parent ComponentR11, child servoR21, origin xyz=0.0 -0.035632 -0.056074 rpy=0 0 0, axis -0.0 0.0 1.0
- added joint Rev70: type continuous, parent servoR31, child ComponentR31Component171, origin xyz=-0.01631 -0.014223 -0.00587 rpy=0 0 0, axis -1.0 0.0 -0.0
- added joint Rev71: type continuous, parent ComponentR31Component171, child ServoR41, origin xyz=0.0 -0.109808 -4.1e-05 rpy=0 0 0, axis 1.0 -0.0 0.0
- added joint Rev72: type continuous, parent ComponentR51Component241, child ServoR61, origin xyz=0.01 -0.034388 -0.018875 rpy=0 0 0, axis -0.0 0.0 -1.0
- added joint Rev73: type continuous, parent ComponentR41, child servoR51, origin xyz=-0.015856 -0.124222 -0.00587 rpy=0 0 0, axis -1.0 0.0 -0.0
- added joint Rev74: type continuous, parent servoL11, child ComponentL11, origin xyz=-0.00587 -0.01631 0.034578 rpy=0 0 0, axis -0.0 -1.0 0.0
- added joint Rev75: type continuous, parent ComponentL11, child ServoL21, origin xyz=0.0 -0.035632 -0.056074 rpy=0 0 0, axis 0.0 0.0 1.0
- added joint Rev76: type continuous, parent servoL31, child ComponentL31Component311, origin xyz=0.03286 0.223131 -0.123204 rpy=0 0 0, axis 1.0 -0.0 0.0
- added joint Rev77: type continuous, parent ComponentL31Component311, child ServoL41, origin xyz=0.0 -0.109809 -4.1e-05 rpy=0 0 0, axis 1.0 -0.0 0.0
- added joint Rev79: type continuous, parent ComponentL51, child ServoL61, origin xyz=-0.01 -0.034388 -0.018875 rpy=0 0 0, axis 0.0 -0.0 1.0
- added joint Rev81: type continuous, parent ComponentL41, child ServoL51, origin xyz=0.015855 -0.124222 0.005874 rpy=0 0 0, axis -1.0 0.0 -0.0
- added joint Rigid80: type fixed, parent ServoL61, child ComponentL61, origin xyz=-0.034577 0.005874 -0.01631 rpy=0 0 0
- added joint Rigid82: type fixed, parent ComponentR21, child servoR31, origin xyz=0.017693 0.008351 0.045045 rpy=0 0 0
- joint Rigid16: child New_comp_v31 -> ComponentR21; origin xyz=-0.033623 -0.026029 0.20616 rpy=0 0 0 -> xyz=-0.034578 0.00587 0.01631 rpy=0 0 0; parent servo_v1_21 -> servoR21
- joint Rigid22: child puru_returns_Component3_Copy_v11 -> ComponentR41; origin xyz=-0.2846 0.036517 0.036019 rpy=0 0 0 -> xyz=0.01631 0.014222 0.00587 rpy=0 0 0; parent servo_v1_51 -> ServoR41
- joint Rigid28: child puru_returns_Component1_v21 -> ComponentR61; origin xyz=-0.007837 -0.000425 -0.424031 rpy=0 0 0 -> xyz=-0.01443 0.403351 -0.020165 rpy=0 0 0; parent servo_v1_71 -> ServoR61
- joint Rigid29: child testing_Component2_Copy_v11Component241 -> ComponentR51Component241; origin xyz=-0.3946 0.064272 -0.01642 rpy=0 0 0 -> xyz=0.01631 0.034577 0.005875 rpy=0 0 0; parent servo_v1_61 -> servoR51
- joint Rigid35: child New_comp_mirror_v11 -> ComponentL21; origin xyz=-0.064468 -0.026024 0.20441 rpy=0 0 0 -> xyz=0.034577 0.005875 0.01631 rpy=0 0 0; parent servo_v1_31 -> ServoL21
- joint Rigid36: child servo_v1_81 -> servoL31; origin xyz=-0.017692 0.00835 0.033301 rpy=0 0 0 -> xyz=-0.034622 -0.229003 0.162375 rpy=0 0 0; parent New_comp_mirror_v11 -> ComponentL21
- joint Rigid40: child puru_returns_Component3_Copy_mirror_v11 -> ComponentL41; origin xyz=-0.314215 0.034762 -0.13273 rpy=0 0 0 -> xyz=-0.01631 0.014222 -0.00587 rpy=0 0 0; parent servo_v1_91 -> ServoL41
- joint Rigid43: child testing_Component2__mirror_v11 -> ComponentL51; parent servo_v1_101 -> ServoL51
- joint Rigid56: child servo_v11 -> servoR1v11; origin xyz=-0.006829 -0.137658 -0.013403 rpy=0 0 0 -> xyz=-0.009829 -0.137658 0.001597 rpy=0 0 0
- joint Rigid57: child servo_v1_11 -> servoL11; origin xyz=0.104916 -0.137658 -0.013403 rpy=0 0 0 -> xyz=0.101916 -0.137658 0.001597 rpy=0 0 0

Commit message: local commit

File: biped_model.urdf (robot description, URDF)
Before this commit: robot COM, 37 links, 36 joints
Joints:
- joint Rev12: limit (none) -> lower=-3.141 upper=3.141 effort=1000 velocity=5; type continuous -> revolute
- joint Rev14: limit (none) -> lower=-3.141 upper=3.141 effort=1000 velocity=5; type continuous -> revolute
- joint Rev18: limit (none) -> lower=-3.141 upper=3.141 effort=1000 velocity=5; type continuous -> revolute
- joint Rev21: limit (none) -> lower=-3.141 upper=3.141 effort=1000 velocity=5; type continuous -> revolute
- joint Rev24: limit (none) -> lower=-3.141 upper=3.141 effort=1000 velocity=5; type continuous -> revolute
- joint Rev27: limit (none) -> lower=-3.141 upper=3.141 effort=1000 velocity=5; type continuous -> revolute
- joint Rev33: limit (none) -> lower=-3.141 upper=3.141 effort=1000 velocity=5; type continuous -> revolute
- joint Rev39: limit (none) -> lower=-3.141 upper=3.141 effort=1000 velocity=5; type continuous -> revolute
- joint Rev42: limit (none) -> lower=-3.141 upper=3.141 effort=1000 velocity=5; type continuous -> revolute
- joint Rev46: limit (none) -> lower=-3.141 upper=3.141 effort=1000 velocity=5; type continuous -> revolute
- joint Rev7: limit (none) -> lower=-3.141 upper=3.141 effort=1000 velocity=5; type continuous -> revolute
- joint Rev8: limit (none) -> lower=-3.141 upper=3.141 effort=1000 velocity=5; type continuous -> revolute

Commit message: fixed motor collapse issue

File: biped_model.urdf (robot description, URDF)
Before this commit: robot biped_model, 25 links, 24 joints
Links:
- link base_link: mass 6.087495213581755 -> 1.087495213581755

Commit message: reorganized code and slighty modified friction

File: biped_model.urdf (robot description, URDF)
Before this commit: robot biped_model, 25 links, 24 joints
Links:
- link ComponentL11: geometry collision mesh filename=meshes/ComponentL11.stl scale=0.001 0.001 0.001; visual mesh filename=meshes/ComponentL11.stl scale=0.001 0.001 0.001
- link ComponentL21: geometry collision mesh filename=meshes/ComponentL21.stl scale=0.001 0.001 0.001; visual mesh filename=meshes/ComponentL21.stl scale=0.001 0.001 0.001
- link ComponentL31Component311: geometry collision mesh filename=meshes/ComponentL31Component311.stl scale=0.001 0.001 0.001; visual mesh filename=meshes/ComponentL31Component311.stl scale=0.001 0.001 0.001
- link ComponentL41: geometry collision mesh filename=meshes/ComponentL41.stl scale=0.001 0.001 0.001; visual mesh filename=meshes/ComponentL41.stl scale=0.001 0.001 0.001
- link ComponentL51: geometry collision mesh filename=meshes/ComponentL51.stl scale=0.001 0.001 0.001; visual mesh filename=meshes/ComponentL51.stl scale=0.001 0.001 0.001
- link ComponentL61: geometry collision mesh filename=meshes/ComponentL61.stl scale=0.001 0.001 0.001; visual mesh filename=meshes/ComponentL61.stl scale=0.001 0.001 0.001
- link ComponentR11: geometry collision mesh filename=meshes/ComponentR11.stl scale=0.001 0.001 0.001; visual mesh filename=meshes/ComponentR11.stl scale=0.001 0.001 0.001
- link ComponentR21: geometry collision mesh filename=meshes/ComponentR21.stl scale=0.001 0.001 0.001; visual mesh filename=meshes/ComponentR21.stl scale=0.001 0.001 0.001
- link ComponentR31Component171: geometry collision mesh filename=meshes/ComponentR31Component171.stl scale=0.001 0.001 0.001; visual mesh filename=meshes/ComponentR31Component171.stl scale=0.001 0.001 0.001
- link ComponentR41: geometry collision mesh filename=meshes/ComponentR41.stl scale=0.001 0.001 0.001; visual mesh filename=meshes/ComponentR41.stl scale=0.001 0.001 0.001
- link ComponentR51Component241: geometry collision mesh filename=meshes/ComponentR51Component241.stl scale=0.001 0.001 0.001; visual mesh filename=meshes/ComponentR51Component241.stl scale=0.001 0.001 0.001
- link ComponentR61: geometry collision mesh filename=meshes/ComponentR61.stl scale=0.001 0.001 0.001; visual mesh filename=meshes/ComponentR61.stl scale=0.001 0.001 0.001
- link ServoL21: geometry collision mesh filename=meshes/ServoL21.stl scale=0.001 0.001 0.001; visual mesh filename=meshes/ServoL21.stl scale=0.001 0.001 0.001
- link ServoL41: geometry collision mesh filename=meshes/ServoL41.stl scale=0.001 0.001 0.001; visual mesh filename=meshes/ServoL41.stl scale=0.001 0.001 0.001
- link ServoL51: geometry collision mesh filename=meshes/ServoL51.stl scale=0.001 0.001 0.001; visual mesh filename=meshes/ServoL51.stl scale=0.001 0.001 0.001
- link ServoL61: geometry collision mesh filename=meshes/ServoL61.stl scale=0.001 0.001 0.001; visual mesh filename=meshes/ServoL61.stl scale=0.001 0.001 0.001
- link ServoR41: geometry collision mesh filename=meshes/ServoR41.stl scale=0.001 0.001 0.001; visual mesh filename=meshes/ServoR41.stl scale=0.001 0.001 0.001
- link ServoR61: geometry collision mesh filename=meshes/ServoR61.stl scale=0.001 0.001 0.001; visual mesh filename=meshes/ServoR61.stl scale=0.001 0.001 0.001
- link base_link: mass 1.087495213581755 -> 1.487495213581755; geometry collision mesh filename=meshes/base_link.stl scale=0.001 0.001 0.001; visual mesh filename=meshes/base_link.stl scale=0.001 0.001 0.001
- link servoL11: geometry collision mesh filename=meshes/servoL11.stl scale=0.001 0.001 0.001; visual mesh filename=meshes/servoL11.stl scale=0.001 0.001 0.001
- link servoL31: geometry collision mesh filename=meshes/servoL31.stl scale=0.001 0.001 0.001; visual mesh filename=meshes/servoL31.stl scale=0.001 0.001 0.001
- link servoR1v11: geometry collision mesh filename=meshes/servoR1v11.stl scale=0.001 0.001 0.001; visual mesh filename=meshes/servoR1v11.stl scale=0.001 0.001 0.001
- link servoR21: geometry collision mesh filename=meshes/servoR21.stl scale=0.001 0.001 0.001; visual mesh filename=meshes/servoR21.stl scale=0.001 0.001 0.001
- link servoR31: geometry collision mesh filename=meshes/servoR31.stl scale=0.001 0.001 0.001; visual mesh filename=meshes/servoR31.stl scale=0.001 0.001 0.001
- link servoR51: geometry collision mesh filename=meshes/servoR51.stl scale=0.001 0.001 0.001; visual mesh filename=meshes/servoR51.stl scale=0.001 0.001 0.001

Commit message: changes foot

File: biped_model.urdf (robot description, URDF)
Before this commit: robot biped_model, 25 links, 24 joints
Links:
- link ComponentL61: mass 0.3521119210080811 -> 0.4041576625809834
- link ComponentR61: mass 0.3521119210080813 -> 0.4039555240314861
Joints:
- removed joint Rigid28
- removed joint Rigid80
- added joint Rigid83: type fixed, parent ServoL61, child ComponentL61, origin xyz=0.014223 0.005874 -0.01631 rpy=0 0 0
- added joint Rigid84: type fixed, parent ServoR61, child ComponentR61, origin xyz=0.034578 0.00587 -0.01631 rpy=0 0 0
