Commit message: adding corrected track

File: track.urdf (robot description, URDF)
Before this commit: robot (Unsaved), 1 links, 0 joints
Links:
- link base_link: geometry collision mesh filename=meshes/base_link_track.stl scale=0.001 0.001 0.001; visual mesh filename=meshes/base_link_track.stl scale=0.001 0.001 0.001

Commit message: added new track

File: track.urdf (robot description, URDF)
Before this commit: robot (Unsaved), 1 links, 0 joints
Links:
- link base_link: mass 105900.920070873599 -> 1376.9212244293362
